File: BC95_NB-IOT.kicad_pcb (KiCad board)
At the start: 4 copper layers, 99.1 x 99.1 mm, 182 parts, among them J1 VIN, J10 Relay_OUT1, J11 Relay_OUT2, J2 USART2, J3 USB_B_Micro, J4 ANALOG_IN, J5 SIM_Card_Shielded, J6 INPUT, J8 Relay_OUT1, J9 Relay_OUT2, K1 ALDP105W, K2 ALDP105W, K3 ALDP105W, K4 ALDP105W, Q11 FDV303N, Q12 FDV303N, Q2 2N7002, Q4 FDV303N, Q5 FDV303N, Q6 Si2301CDS, Q8 FDV303N, Q9 FDV303N, SW1 RESET, U1 SHT4x, U2 TPS54331DDA, U3 STM32L051K6Tx, U4 QUECTEL_BG96, U5 AMS1117CD-3.3, U6 ULN2003A, U7 FOD817ASD, U8 FOD817ASD, U9 LM1085-ADJ

Commit message: Add files via upload
Parts:
- moved C5 0.48 mm to (74.8, 33.9)
- moved C8 0.42 mm to (82.0, 119.0)
- moved C3 0.37 mm to (82.0, 121.5)
- moved Q6 0.33 mm to (69.3, 64.8)
- moved R13 0.17 mm to (86.0, 79.0)
- moved R32 0.16 mm to (64.6, 64.6)
- moved R31 0.15 mm to (66.2, 64.6)
- moved R66 0.13 mm to (81.5, 83.0)
- moved R64 0.08 mm to (83.3, 83.1)
- moved R12 0.08 mm to (87.5, 79.0)
- moved D30 0.06 mm to (85.2, 83.1)
Connections:
- D15 pad 1: GND -> GNDA
- D16 pad 1: GND -> GNDA
- J6 pad 2: GND -> GNDA
- U7 pad 1: +3V3 -> Net-(R25-Pad2)
- U7 pad 2: V_IN1 -> GNDA
- U7 pad 3: GND -> V_IN1
- U7 pad 4: Net-(R25-Pad2) -> +3V3
- U8 pad 2: GND -> GNDA
Routing:
- net MODULE_UART_TX: track 0.00 -> 55.1 mm, vias 0 -> 2
- net GNDA: track 0.00 -> 37.1 mm, vias 0 -> 2
- net MODULE_UART_RX: track 71.9 -> 101.0 mm, vias 2 -> 3
- net Net-(R66-Pad2): track 0.00 -> 26.3 mm, vias 0 -> 2
- net +6V: track 144.9 -> 166.7 mm, vias 18 -> 20
- net Net-(J8-Pad1): track 20.2 -> 0.00 mm
- net Net-(J9-Pad1): track 19.9 -> 0.00 mm
- net Net-(J10-Pad1): track 19.8 -> 0.00 mm
- net Net-(J11-Pad1): track 19.4 -> 0.00 mm
- net GND: track 0.30 -> 17.6 mm, vias 0 -> 37
- net Net-(J9-Pad2): track 11.9 -> 0.00 mm
- net Net-(J8-Pad2): track 11.8 -> 0.00 mm
- net Net-(J10-Pad2): track 11.6 -> 0.00 mm
- net Net-(J11-Pad2): track 11.2 -> 0.00 mm
- net W_DISABLE: track 0.00 -> 11.1 mm
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- added copper zone on B.Cu, net GND
- added copper zone on F.Cu, net GND
- added copper zone on In2.Cu, net GND
- added copper zone on B.Cu, net Net-(J10-Pad1)
- added copper zone on F.Cu, net Net-(J10-Pad2)
- added copper zone on B.Cu, net Net-(J11-Pad1)
- added copper zone on F.Cu, net Net-(J11-Pad2)
- added copper zone on B.Cu, net Net-(J8-Pad1)
- added copper zone on F.Cu, net Net-(J8-Pad2)
- added copper zone on B.Cu, net Net-(J9-Pad1)
- added copper zone on F.Cu, net Net-(J9-Pad2)
- removed copper zone on In2.Cu, net (none)
Other:
- outline, holes or cut-outs redrawn

Commit message: bom update
Parts:
- removed the REF** at (-90.6, -18.5)
- removed the REF** at (-99.2, -15.7)
- added G***: LOGO, LOGO, F.Cu at (106.7, 137.7)
- AE1, AE2: footprint Connector_Coaxial:SMA_Amphenol_901-144_Vertical -> Connector_Coaxial:SMA_Amphenol_132134-10_Vertical
- H1, H2, H3, H4: footprint MountingHole:MountingHole_3.2mm_M3_Pad_Via -> MountingHole:MountingHole_3.2mm_M3_Pad
- J1: footprint TerminalBlock_Altech:Altech_AK300_1x02_P5.00mm_45-Degree -> TerminalBlock_Phoenix:TerminalBlock_Phoenix_MKDS-1,5-2-5.08_1x02_P5.08mm_Horizontal
- J10, J11, J8, J9: footprint TerminalBlock_Altech:Altech_AK300_1x02_P5.00mm_45-Degree -> Connector_Phoenix_MC_HighVoltage:PhoenixContact_MC_1,5_2-G-5.08_1x02_P5.08mm_Horizontal
- REF**: moved to B.Cu
- moved REF** 178.5 mm to (53.8, 81.0), turned to 60 degrees
- moved C5 2.87 mm to (72.0, 34.4)
- moved U1 2.50 mm to (72.4, 36.8)
- moved C10 2.28 mm to (75.2, 38.0), turned to 0 degrees
- moved R6 1.58 mm to (74.3, 40.3)
- moved J1 1.56 mm to (67.4, 38.6)
- moved R7 1.47 mm to (72.4, 40.2)
- moved FB2 0.34 mm to (59.2, 83.5)
- moved R61 0.28 mm to (108.0, 115.7)
- moved D29 0.25 mm to (108.0, 114.0)
- moved C45 0.15 mm to (57.6, 61.5)
- moved D17 0.05 mm to (62.1, 121.4)
- turned AE1 to 90 degrees
Routing:
- net Net-(C19-Pad1): track 77.5 -> 40.5 mm, vias 6 -> 7
- net Net-(C39-Pad1): track 8.01 -> 0.17 mm
- net GND: track 17.6 -> 22.2 mm, vias 37 -> 367
- net +3V3: track 156.2 -> 153.2 mm
- net Net-(R7-Pad2): track 37.5 -> 35.8 mm
- net MODULE_UART_RX: track 101.0 -> 99.3 mm
- net Net-(D10-Pad2): track 13.3 -> 14.9 mm
- net +6V: track 166.7 -> 166.0 mm
- added copper zone on F.Cu, net Net-(C39-Pad1)
Other:
- board text added: "AIN"
- board text added: "DIN"
- board text added: "GNSS"
- board text added: "H. YUCEL COGAL"
- board text added: "HYC"
- board text added: "LPWAN & NB-IoT REMOTE CONTROL & MONITOR"
- board text added: "MAIN"
- board text added: "OUT1"
- board text added: "OUT2"
- board text added: "OUT3"
- board text added: "OUT4"
- board text added: "RST"
- board text added: "SIM"
- board text added: "SWD"
- board text added: "USB"
- board text added: "VIN"

Commit message: Add files via upload
Parts:
- AE1, AE2: value Antenna_Shield -> (none)
- C12, C2, C7: footprint Capacitor_SMD:C_1206_3216Metric_Pad1.33x1.80mm_HandSolder -> Capacitor_SMD:C_1206_3216Metric
- C14, C16, C17, C18, C26, C45: footprint Capacitor_SMD:C_0603_1608Metric_Pad1.08x0.95mm_HandSolder -> Capacitor_SMD:C_0603_1608Metric
- C28, C31, C33: footprint Capacitor_Tantalum_SMD:CP_EIA-3528-21_Kemet-B_Pad1.50x2.35mm_HandSolder -> Capacitor_Tantalum_SMD:CP_EIA-3528-21_Kemet-B
- D1: value CDBA340-HF -> B350-A-13-F
- D22, D25, D6: value TZMC5V1 -> BZV55-C6V2,115
- Q6: value Si2301CDS -> DMG2305UX-7
- R19, R20, R4, R5, R8: footprint Resistor_SMD:R_0603_1608Metric_Pad0.98x0.95mm_HandSolder -> Resistor_SMD:R_0603_1608Metric
- R66: value 0r (DNP) -> 0R(DNI)
- turned C28 to 0 degrees
- turned C31 to -90 degrees
- turned C33 to -90 degrees
Connections:
- C28 pad 1: GND -> +6V
- C28 pad 2: +6V -> GND
- C31 pad 1: GND -> +6V
- C31 pad 2: +6V -> GND
- C33 pad 1: GND -> +6V
- C33 pad 2: +6V -> GND
