File: BC95_NB-IOT.kicad_sch (KiCad schematic)
At the start: 179 parts, among them J1 VIN, J10 Relay_OUT1, J11 Relay_OUT2, J2 USART2, J3 USB_B_Micro, J4 ANALOG_IN, J5 SIM_Card_Shielded, J6 INPUT, J8 Relay_OUT1, J9 Relay_OUT2, K1 ALDP105W, K2 ALDP105W, K3 ALDP105W, K4 ALDP105W, Q11 FDV303N, Q12 FDV303N, Q2 2N7002, Q4 FDV303N, Q5 FDV303N, Q6 Si2301CDS, Q8 FDV303N, Q9 FDV303N, SW1 RESET, U1 SHT4x, U2 TPS54331DDA, U3 STM32L051K6Tx, U4 QUECTEL_BG96, U5 AMS1117CD-3.3, U6 ULN2003A, U7 FOD817ASD, U8 FOD817ASD, U9 LM1085-ADJ

Commit message: Add files via upload
Connections:
- net +3V3: now also U7.4; no longer U7.1
- net GND: no longer D15.1 (A1), D16.1 (A1), J6.2 (Pin_2), U7.3, U8.2
- net V_IN1: now also U7.3; no longer U7.2
- net at R25.2: now also U7.1; no longer U7.4
- new net GNDA: D15.1 (A1), D16.1 (A1), J6.2 (Pin_2), U7.2, U8.2
Changed lines of the file:
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@@
     (pin "1")
   )
-  (symbol (lib_id "power:GND") (at 514.35 97.79 0) (mirror y) (unit 1)
-    (in_bom yes) (on_board yes) (fields_autoplaced)
-    (property "Reference" "#PWR0141" (id 0) (at 514.35 104.14 0)
-      (effects (font (size 1.27 1.27)) hide)
-    )
-    (property "Value" "GND" (id 1) (at 514.35 102.87 0))
-    (property "Footprint" "" (id 2) (at 514.35 97.79 0)
-      (effects (font (size 1.27 1.27)) hide)
-    )
-    (property "Datasheet" "" (id 3) (at 514.35 97.79 0)
-      (effects (font (size 1.27 1.27)) hide)
-    )
-    (pin "1")
-  )
   (symbol (lib_id "power:GND") (at 133.35 73.66 0) (unit 1)
     (in_bom yes) (on_board yes)
@@
     (pin "2")
   )
-  (symbol (lib_id "power:GND") (at 551.18 129.54 0) (unit 1)
-    (in_bom yes) (on_board yes) (fields_autoplaced)
-    (property "Reference" "#PWR0146" (id 0) (at 551.18 135.89 0)
-      (effects (font (size 1.27 1.27)) hide)
-    )
-    (property "Value" "GND" (id 1) (at 551.18 134.62 0))
-    (property "Footprint" "" (id 2) (at 551.18 129.54 0)
-      (effects (font (size 1.27 1.27)) hide)
-    )
-    (property "Datasheet" "" (id 3) (at 551.18 129.54 0)
-      (effects (font (size 1.27 1.27)) hide)
-    )
-    (pin "1")
-  )
   (symbol (lib_id "Device:Fuse") (at 50.8 43.18 90) (unit 1)
     (in_bom yes) (on_board yes) (fields_autoplaced)
@@
     (pin "1")
   )
-  (symbol (lib_id "power:GND") (at 471.17 114.3 0) (unit 1)
-    (in_bom yes) (on_board yes) (fields_autoplaced)
-    (property "Reference" "#PWR0201" (id 0) (at 471.17 120.65 0)
-      (effects (font (size 1.27 1.27)) hide)
-    )
-    (property "Value" "GND" (id 1) (at 471.17 119.38 0))
-    (property "Footprint" "" (id 2) (at 471.17 114.3 0)
-      (effects (font (size 1.27 1.27)) hide)
-    )
-    (property "Datasheet" "" (id 3) (at 471.17 114.3 0)
-      (effects (font (size 1.27 1.27)) hide)
-    )
-    (pin "1")
-  )
   (symbol (lib_id "Device:C_Small") (at 139.7 255.27 0) (unit 1)
     (in_bom yes) (on_board yes)
@@
     (pin "2")
   )
+  (symbol (lib_id "power:GNDA") (at 471.17 114.3 0) (unit 1)
+    (in_bom yes) (on_board yes) (fields_autoplaced)
+    (property "Reference" "#PWR0127" (id 0) (at 471.17 120.65 0)
+      (effects (font (size 1.27 1.27)) hide)
+    )
+    (property "Value" "GNDA" (id 1) (at 471.17 119.38 0))
+    (property "Footprint" "" (id 2) (at 471.17 114.3 0)
+      (effects (font (size 1.27 1.27)) hide)
+    )
+    (property "Datasheet" "" (id 3) (at 471.17 114.3 0)
+      (effects (font (size 1.27 1.27)) hide)
+    )
+    (pin "1")
+  )
   (symbol (lib_id "power:GND") (at 111.76 199.39 0) (unit 1)
     (in_bom yes) (on_board yes)
@@
     (pin "2")
   )
+  (symbol (lib_id "power:GNDA") (at 514.35 97.79 0) (unit 1)
+    (in_bom yes) (on_board yes) (fields_autoplaced)
+    (property "Reference" "#PWR0125" (id 0) (at 514.35 104.14 0)
+      (effects (font (size 1.27 1.27)) hide)
+    )
+    (property "Value" "GNDA" (id 1) (at 514.35 102.87 0))
+    (property "Footprint" "" (id 2) (at 514.35 97.79 0)
+      (effects (font (size 1.27 1.27)) hide)
+    )
+    (property "Datasheet" "" (id 3) (at 514.35 97.79 0)
+      (effects (font (size 1.27 1.27)) hide)
+    )
+    (pin "1")
+  )
   (symbol (lib_id "power:GND") (at 196.85 198.12 0) (unit 1)
     (in_bom yes) (on_board yes)
@@
     (pin "2")
   )
+  (symbol (lib_id "power:GNDA") (at 551.18 129.54 0) (unit 1)
+    (in_bom yes) (on_board yes) (fields_autoplaced)
+    (property "Reference" "#PWR0103" (id 0) (at 551.18 135.89 0)
+      (effects (font (size 1.27 1.27)) hide)
+    )
+    (property "Value" "GNDA" (id 1) (at 551.18 134.62 0))
+    (property "Footprint" "" (id 2) (at 551.18 129.54 0)
+      (effects (font (size 1.27 1.27)) hide)
+    )
+    (property "Datasheet" "" (id 3) (at 551.18 129.54 0)
+      (effects (font (size 1.27 1.27)) hide)
+    )
+    (pin "1")
+  )
   (symbol (lib_id "Device:R_Small") (at 334.01 218.44 0) (unit 1)
     (in_bom yes) (on_board yes) (fields_autoplaced)
@@
     (pin "2")
   )
+  (symbol (lib_id "power:GNDA") (at 478.79 129.54 0) (unit 1)
+    (in_bom yes) (on_board yes) (fields_autoplaced)
+    (property "Reference" "#PWR0128" (id 0) (at 478.79 135.89 0)
+      (effects (font (size 1.27 1.27)) hide)
+    )
+    (property "Value" "GNDA" (id 1) (at 478.79 134.62 0))
+    (property "Footprint" "" (id 2) (at 478.79 129.54 0)
+      (effects (font (size 1.27 1.27)) hide)
+    )
+    (property "Datasheet" "" (id 3) (at 478.79 129.54 0)
+      (effects (font (size 1.27 1.27)) hide)
+    )
+    (pin "1")
+  )
   (symbol (lib_id "power:GND") (at 214.63 229.87 0) (unit 1)
     (in_bom yes) (on_board yes)
@@
     (pin "1")
   )
+  (symbol (lib_id "power:GNDA") (at 558.8 114.3 0) (unit 1)
+    (in_bom yes) (on_board yes) (fields_autoplaced)
+    (property "Reference" "#PWR0116" (id 0) (at 558.8 120.65 0)
+      (effects (font (size 1.27 1.27)) hide)
+    )
+    (property "Value" "GNDA" (id 1) (at 558.8 119.38 0))
+    (property "Footprint" "" (id 2) (at 558.8 114.3 0)
+      (effects (font (size 1.27 1.27)) hide)
+    )
+    (property "Datasheet" "" (id 3) (at 558.8 114.3 0)
+      (effects (font (size 1.27 1.27)) hide)
+    )
+    (pin "1")
+  )
   (symbol (lib_id "Device:R_Small") (at 130.81 238.76 270) (unit 1)
     (in_bom yes) (on_board yes)
@@
     (pin "1")
   )
-  (symbol (lib_id "power:GND") (at 558.8 114.3 0) (unit 1)
-    (in_bom yes) (on_board yes) (fields_autoplaced)
-    (property "Reference" "#PWR0200" (id 0) (at 558.8 120.65 0)
-      (effects (font (size 1.27 1.27)) hide)
-    )
-    (property "Value" "GND" (id 1) (at 558.8 119.38 0))
-    (property "Footprint" "" (id 2) (at 558.8 114.3 0)
-      (effects (font (size 1.27 1.27)) hide)
-    )
-    (property "Datasheet" "" (id 3) (at 558.8 114.3 0)
-      (effects (font (size 1.27 1.27)) hide)
-    )
-    (pin "1")
-  )
   (symbol (lib_id "Device:D_Zener") (at 219.71 193.04 270) (unit 1)
     (in_bom yes) (on_board yes) (fields_autoplaced)
@@
     (pin "1")
   )
-  (symbol (lib_id "power:GND") (at 478.79 129.54 0) (mirror y) (unit 1)
-    (in_bom yes) (on_board yes) (fields_autoplaced)
-    (property "Reference" "#PWR0145" (id 0) (at 478.79 135.89 0)
-      (effects (font (size 1.27 1.27)) hide)
-    )
-    (property "Value" "GND" (id 1) (at 478.79 134.62 0))
-    (property "Footprint" "" (id 2) (at 478.79 129.54 0)
-      (effects (font (size 1.27 1.27)) hide)
-    )
-    (property "Datasheet" "" (id 3) (at 478.79 129.54 0)
-      (effects (font (size 1.27 1.27)) hide)
-    )
-    (pin "1")
-  )
   (symbol (lib_id "power:+3.3V") (at 69.85 153.67 0) (unit 1)
     (in_bom yes) (on_board yes) (fields_autoplaced)
@@
     (pin "1")
   )
-  (symbol (lib_id "Isolator:LTV-817S") (at 492.76 118.11 0) (mirror y) (unit 1)
+  (symbol (lib_id "Isolator:LTV-817S") (at 492.76 118.11 0) (unit 1)
     (in_bom yes) (on_board yes) (fields_autoplaced)
     (property "Reference" "U7" (id 0) (at 492.76 109.22 0))
@@
       (effects (font (size 1.27 1.27)) hide)
     )
-    (property "Datasheet" "https://ozdisan.com/optoelectronics-and-sensors/optoelectronics/optocoupler-transistor-output/FOD817ASD" (id 3) (at 501.65 110.49 0)
+    (property "Datasheet" "https://ozdisan.com/optoelectronics-and-sensors/optoelectronics/optocoupler-transistor-output/FOD817ASD" (id 3) (at 483.87 110.49 0)
       (effects (font (size 1.27 1.27)) hide)
     )
@@
       (reference "#PWR0102") (unit 1) (value "+6V") (footprint "")
     )
+    (path "/a9bfd587-1c43-4fe5-84ee-8c67c512032f"
+      (reference "#PWR0103") (unit 1) (value "GNDA") (footprint "")
+    )
     (path "/158d2b4a-9469-460b-88d0-735f7b274359"
       (reference "#PWR0104") (unit 1) (value "GND") (footprint "")
@@
       (reference "#PWR0115") (unit 1) (value "+3.3V") (footprint "")
     )
+    (path "/bae57fbf-bcc6-4c5a-a3a2-6909fba5dbf8"
+      (reference "#PWR0116") (unit 1) (value "GNDA") (footprint "")
+    )
     (path "/0a518aaa-f003-43ed-bd0f-68890f4baccc"
       (reference "#PWR0117") (unit 1) (value "GND") (footprint "")
@@
       (reference "#PWR0124") (unit 1) (value "GND") (footprint "")
     )
+    (path "/9285d487-7076-4a48-9acc-31bfec3016f8"
+      (reference "#PWR0125") (unit 1) (value "GNDA") (footprint "")
+    )
     (path "/d73061c4-54a6-44eb-afb1-5af7f2c9c482"
       (reference "#PWR0126") (unit 1) (value "+3V8") (footprint "")
     )
+    (path "/7f0abcb7-39e1-4cbc-8b36-b751fe57a861"
+      (reference "#PWR0127") (unit 1) (value "GNDA") (footprint "")
+    )
+    (path "/b21012d8-d78c-4fd1-8353-8735875c5545"
+      (reference "#PWR0128") (unit 1) (value "GNDA") (footprint "")
+    )
     (path "/af1fe446-8a7b-4b1c-bc06-e2753cd2a734"
       (reference "#PWR0129") (unit 1) (value "GND") (footprint "")
@@
       (reference "#PWR0140") (unit 1) (value "GND") (footprint "")
     )
-    (path "/342e8ca1-802e-47a6-be03-42140b6988de"
-      (reference "#PWR0141") (unit 1) (value "GND") (footprint "")
-    )
     (path "/a2066b42-2cff-4fdc-83c8-30794098b961"
       (reference "#PWR0143") (unit 1) (value "+3.3V") (footprint "")
@@
       (reference "#PWR0144") (unit 1) (value "GND") (footprint "")
     )
-    (path "/df5efdbd-71c2-48e1-ae7d-1b82ddcabeef"
-      (reference "#PWR0145") (unit 1) (value "GND") (footprint "")
-    )
-    (path "/4c8e0e49-119f-4514-a8fe-be53da85ce88"
-      (reference "#PWR0146") (unit 1) (value "GND") (footprint "")
-    )
     (path "/0853e952-c923-45ed-8b81-8249c50f2dd9"
       (reference "#PWR0147") (unit 1) (value "GND") (footprint "")
@@
       (reference "#PWR0199") (unit 1) (value "GND") (footprint "")
     )
-    (path "/c2fb4485-b319-45e8-b836-b9e67bcac56c"
-      (reference "#PWR0200") (unit 1) (value "GND") (footprint "")
-    )
-    (path "/69d62dd2-e26f-4f1c-9904-b3153e7eea7f"
-      (reference "#PWR0201") (unit 1) (value "GND") (footprint "")
-    )
     (path "/c08ec128-354c-44fd-8603-24fe20b0fb01"

Commit message: bom update
Parts:
- AE1, AE2: footprint Connector_Coaxial:SMA_Amphenol_901-144_Vertical -> Connector_Coaxial:SMA_Amphenol_132134-10_Vertical
- C28, C31, C33: footprint Capacitor_Tantalum_SMD:CP_EIA-3528-21_Kemet-B_Pad1.50x2.35mm_HandSolder -> Capacitor_Tantalum_SMD:CP_EIA-3528-21_Kemet-B
- D1: value CDBA340-HF -> B350-A-13-F
- D22, D25, D6: value TZMC5V1 -> BZV55-C6V2,115
- H1, H2, H3, H4: footprint MountingHole:MountingHole_3.2mm_M3_Pad_Via -> MountingHole:MountingHole_3.2mm_M3_Pad
- J1: footprint TerminalBlock_Altech:Altech_AK300_1x02_P5.00mm_45-Degree -> TerminalBlock_Phoenix:TerminalBlock_Phoenix_MKDS-1,5-2-5.08_1x02_P5.08mm_Horizontal
- J10, J11, J8, J9: footprint TerminalBlock_Altech:Altech_AK300_1x02_P5.00mm_45-Degree -> Connector_Phoenix_MC_HighVoltage:PhoenixContact_MC_1,5_2-G-5.08_1x02_P5.08mm_Horizontal
- Q6: value Si2301CDS -> DMG2305UX-7
Other:
- note removed: "ULN2003A KOY"
- moved on the sheet: C54, H1, H2, H3, H4, J2

Commit message: Add files via upload
Parts:
- AE1, AE2: value Antenna_Shield -> (none); STANDART (none) -> x
- C1, C10, C11, C13, C15, C19, C20, C21, C22, C23, C24, C25, C27, C28, C29, C31, C32, C33, C34, C35, C36, C37, C38, C39, C40, C41, C42, C43, C44, C46, C47, C48, C49, C5, C50, C51, C52, C53, C54, C6, D1, D10, D11, D12, D13, D14, D15, D16, D17, D18, D19, D2, D22, D23, D24, D25, D26, D29, D3, D30, D4, D5, D6, D7, D8, D9, F1, FB1, FB2, H1, H2, H3, H4, J1, J10, J11, J2, J3, J4, J5, J6, J8, J9, L1, Q11, Q12, Q2, Q4, Q5, Q6, Q8, Q9, R1, R10, R11, R12, R13, R14, R15, R16, R17, R18, R2, R24, R25, R26, R29, R3, R30, R31, R32, R33, R34, R35, R36, R37, R38, R39, R40, R41, R42, R44, R45, R46, R48, R49, R50, R51, R52, R53, R54, R55, R56, R57, R58, R6, R61, R64, R65, R67, R68, R7, R9, SW1, SWD1, U2, U3, U5, U6, U7, U8, U9: STANDART (none) -> x
- C12, C2, C7: footprint Capacitor_SMD:C_1206_3216Metric_Pad1.33x1.80mm_HandSolder -> Capacitor_SMD:C_1206_3216Metric; STANDART (none) -> x
- C14, C16, C17, C18, C26, C45: footprint Capacitor_SMD:C_0603_1608Metric_Pad1.08x0.95mm_HandSolder -> Capacitor_SMD:C_0603_1608Metric; STANDART (none) -> x
- K1, K2, K3, K4: STANDART Manufacturer Recommendations -> x
- R19, R20, R4, R5, R8: footprint Resistor_SMD:R_0603_1608Metric_Pad0.98x0.95mm_HandSolder -> Resistor_SMD:R_0603_1608Metric; STANDART (none) -> x
- R66: value 0r (DNP) -> 0R(DNI); STANDART (none) -> x
Connections:
- net +6V: now also C28.1, C31.1, C33.1; no longer C28.2, C31.2, C33.2
- net GND: now also C28.2, C31.2, C33.2; no longer C28.1, C31.1, C33.1
Other:
- moved on the sheet: C28, C31, C33, D11, D12, D26, D29, J10, J11, J8, J9, K1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
